File: Design Files/NB-IoT-ideaboard-v2.0.brd (EAGLE design)
At the start: 93 x 65 mm, 120 parts, among them Q1 32.768kHz, Q2 9013, Q3 9013, Q4 9013, Q5 9013, U1 STM32F103RBT6, U2 MCP73831T-2ACI/OT, U3 AP2112-3.3, U4 PAM2401, U5 MICROSIM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

Commit message: Finalizing manufacturing files and 3D model
Routing:
- net GND: vias 150 -> 274
Other:
- board text removed: "add more vias"
- board text removed: "added new components. update BoM"

Commit message: Changes to BoM
Parts:
- C10, C11: value 30pF -> 25pF
- C29, C31: value 100nF -> DNP
- R10: value 0R -> 1k
- R9: value 0R -> 400R
Changed lines of the file:
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@@
 <setting verticaltext="up"/>
 </settings>
-<grid distance="8" unitdist="mil" unit="mil" style="lines" multiple="1" display="no" altdistance="1" altunitdist="mil" altunit="mil"/>
+<grid distance="8" unitdist="mil" unit="mil" style="lines" multiple="1" display="yes" altdistance="1" altunitdist="mil" altunit="mil"/>
 <layers>
 <layer number="1" name="Top" color="4" fill="1" visible="yes" active="yes"/>
@@
 <attribute name="VALUE" x="40.5384" y="54.9148" size="1.27" layer="27" rot="R270"/>
 </element>
-<element name="C10" library="rcl" library_urn="urn:adsk.eagle:library:334" package="C0805" package3d_urn="urn:adsk.eagle:package:23617/2" value="30pF" x="46.1264" y="53.6448" smashed="yes" rot="R270">
+<element name="C10" library="rcl" library_urn="urn:adsk.eagle:library:334" package="C0805" package3d_urn="urn:adsk.eagle:package:23617/2" value="25pF" x="46.1264" y="53.6448" smashed="yes" rot="R270">
 <attribute name="NAME" x="45.466" y="55.3212" size="0.889" layer="25"/>
 <attribute name="SPICEPREFIX" value="C" x="46.1264" y="53.6448" size="1.778" layer="27" rot="R270" display="off"/>
 <attribute name="VALUE" x="43.5864" y="54.9148" size="1.27" layer="27" rot="R270"/>
 </element>
-<element name="C11" library="rcl" library_urn="urn:adsk.eagle:library:334" package="C0805" package3d_urn="urn:adsk.eagle:package:23617/2" value="30pF" x="55.4736" y="53.848" smashed="yes" rot="R270">
+<element name="C11" library="rcl" library_urn="urn:adsk.eagle:library:334" package="C0805" package3d_urn="urn:adsk.eagle:package:23617/2" value="25pF" x="55.4736" y="53.848" smashed="yes" rot="R270">
 <attribute name="NAME" x="56.7436" y="55.118" size="0.889" layer="25" rot="R270"/>
 <attribute name="SPICEPREFIX" value="C" x="55.4736" y="53.848" size="1.778" layer="27" rot="R270" display="off"/>
 <attribute name="VALUE" x="52.9336" y="55.118" size="1.27" layer="27" rot="R270"/>
 </element>
-<element name="R9" library="rcl" library_urn="urn:adsk.eagle:library:334" package="R0805" package3d_urn="urn:adsk.eagle:package:23553/2" value="0R" x="39.8272" y="57.0992" smashed="yes" rot="R180">
+<element name="R9" library="rcl" library_urn="urn:adsk.eagle:library:334" package="R0805" package3d_urn="urn:adsk.eagle:package:23553/2" value="400R" x="39.8272" y="57.0992" smashed="yes" rot="R180">
 <attribute name="NAME" x="39.6494" y="58.8772" size="0.889" layer="25" rot="R180"/>
 <attribute name="SPICEPREFIX" value="R" x="39.8272" y="57.0992" size="1.778" layer="27" rot="R180" display="off"/>
 <attribute name="VALUE" x="40.4622" y="59.6392" size="1.27" layer="27" rot="R180"/>
 </element>
-<element name="R10" library="rcl" library_urn="urn:adsk.eagle:library:334" package="R0805" package3d_urn="urn:adsk.eagle:package:23553/2" value="0R" x="51.0032" y="57.7088" smashed="yes" rot="R180">
+<element name="R10" library="rcl" library_urn="urn:adsk.eagle:library:334" package="R0805" package3d_urn="urn:adsk.eagle:package:23553/2" value="1k" x="51.0032" y="57.7088" smashed="yes" rot="R180">
 <attribute name="NAME" x="48.4124" y="59.1566" size="0.889" layer="25" rot="R270"/>
 <attribute name="SPICEPREFIX" value="R" x="51.0032" y="57.7088" size="1.778" layer="27" rot="R180" display="off"/>
@@
 <attribute name="VALUE" x="76.0984" y="84.7598" size="1.27" layer="27" rot="R270"/>
 </element>
-<element name="C29" library="rcl" library_urn="urn:adsk.eagle:library:334" package="C0805" package3d_urn="urn:adsk.eagle:package:23617/2" value="100nF" x="81.4832" y="83.312" smashed="yes" rot="R180">
+<element name="C29" library="rcl" library_urn="urn:adsk.eagle:library:334" package="C0805" package3d_urn="urn:adsk.eagle:package:23617/2" value="DNP" x="81.4832" y="83.312" smashed="yes" rot="R180">
 <attribute name="NAME" x="83.3628" y="84.1756" size="0.889" layer="25" font="vector" rot="R270"/>
 <attribute name="SPICEPREFIX" value="C" x="81.4832" y="83.312" size="1.778" layer="27" rot="R180" display="off"/>
 <attribute name="VALUE" x="82.7532" y="85.852" size="1.27" layer="27" rot="R180"/>
 </element>
-<element name="C31" library="rcl" library_urn="urn:adsk.eagle:library:334" package="C0805" package3d_urn="urn:adsk.eagle:package:23617/2" value="100nF" x="81.4832" y="85.344" smashed="yes" rot="R180">
+<element name="C31" library="rcl" library_urn="urn:adsk.eagle:library:334" package="C0805" package3d_urn="urn:adsk.eagle:package:23617/2" value="DNP" x="81.4832" y="85.344" smashed="yes" rot="R180">
 <attribute name="NAME" x="83.3628" y="86.614" size="0.889" layer="25" font="vector" rot="R270"/>
 <attribute name="SPICEPREFIX" value="C" x="81.4832" y="85.344" size="1.778" layer="27" rot="R180" display="off"/>

Commit message: Crystal RC values updated. New pcb images added
Parts:
- C10, C11: value 25pF -> 20pF
- R9: value 400R -> 330k
Changed lines of the file:
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@@
 <attribute name="VALUE" x="40.5384" y="54.9148" size="1.27" layer="27" rot="R270"/>
 </element>
-<element name="C10" library="rcl" library_urn="urn:adsk.eagle:library:334" package="C0805" package3d_urn="urn:adsk.eagle:package:23617/2" value="25pF" x="46.1264" y="53.6448" smashed="yes" rot="R270">
+<element name="C10" library="rcl" library_urn="urn:adsk.eagle:library:334" package="C0805" package3d_urn="urn:adsk.eagle:package:23617/2" value="20pF" x="46.1264" y="53.6448" smashed="yes" rot="R270">
 <attribute name="NAME" x="45.466" y="55.3212" size="0.889" layer="25"/>
 <attribute name="SPICEPREFIX" value="C" x="46.1264" y="53.6448" size="1.778" layer="27" rot="R270" display="off"/>
 <attribute name="VALUE" x="43.5864" y="54.9148" size="1.27" layer="27" rot="R270"/>
 </element>
-<element name="C11" library="rcl" library_urn="urn:adsk.eagle:library:334" package="C0805" package3d_urn="urn:adsk.eagle:package:23617/2" value="25pF" x="55.4736" y="53.848" smashed="yes" rot="R270">
+<element name="C11" library="rcl" library_urn="urn:adsk.eagle:library:334" package="C0805" package3d_urn="urn:adsk.eagle:package:23617/2" value="20pF" x="55.4736" y="53.848" smashed="yes" rot="R270">
 <attribute name="NAME" x="56.7436" y="55.118" size="0.889" layer="25" rot="R270"/>
 <attribute name="SPICEPREFIX" value="C" x="55.4736" y="53.848" size="1.778" layer="27" rot="R270" display="off"/>
 <attribute name="VALUE" x="52.9336" y="55.118" size="1.27" layer="27" rot="R270"/>
 </element>
-<element name="R9" library="rcl" library_urn="urn:adsk.eagle:library:334" package="R0805" package3d_urn="urn:adsk.eagle:package:23553/2" value="400R" x="39.8272" y="57.0992" smashed="yes" rot="R180">
+<element name="R9" library="rcl" library_urn="urn:adsk.eagle:library:334" package="R0805" package3d_urn="urn:adsk.eagle:package:23553/2" value="330k" x="39.8272" y="57.0992" smashed="yes" rot="R180">
 <attribute name="NAME" x="39.6494" y="58.8772" size="0.889" layer="25" rot="R180"/>
 <attribute name="SPICEPREFIX" value="R" x="39.8272" y="57.0992" size="1.778" layer="27" rot="R180" display="off"/>
